File: CBC2.kicad_pcb (KiCad board)
At the start: 2 copper layers, 215 parts, among them K0:0 KEYSW, K0:1 KEYSW, K0:10 KEYSW, K0:11 KEYSW, K0:12 KEYSW, K0:13 KEYSW, K0:14 KEYSW, K0:15 KEYSW, K0:16 KEYSW, K0:2 KEYSW, K0:3 KEYSW, K0:4 KEYSW, K0:5 KEYSW, K0:6 KEYSW, K0:7 KEYSW, K0:8 KEYSW, K0:9 KEYSW, K1:0 KEYSW, K1:1 KEYSW, K1:10 KEYSW, K1:11 KEYSW, K1:12 KEYSW, K1:13 KEYSW, K1:14 KEYSW, K1:15 KEYSW, K1:16 KEYSW, K1:17 KEYSW, K1:2 KEYSW, K1:3 KEYSW, K1:4 KEYSW, K1:5 KEYSW, K1:6 KEYSW, K1:7 KEYSW, K1:8 KEYSW, K1:9 KEYSW, K2:0 KEYSW, K2:1 KEYSW, K2:10 KEYSW, K2:11 KEYSW, K2:12 KEYSW, K2:13 KEYSW, K2:14 KEYSW, K2:15 KEYSW, K2:16 KEYSW, K2:17 KEYSW, K2:2 KEYSW, K2:3 KEYSW, K2:4 KEYSW, K2:5 KEYSW, K2:6 KEYSW, K2:7 KEYSW, K2:8 KEYSW, K2:9 KEYSW, K3:0 KEYSW, K3:1 KEYSW, K3:10 KEYSW, K3:11 KEYSW, K3:12 KEYSW, K3:14 KEYSW, K3:15 KEYSW, K3:16 KEYSW, K3:17 KEYSW, K3:2 KEYSW, K3:3 KEYSW, K3:4 KEYSW, K3:5 KEYSW, K3:6 KEYSW, K3:7 KEYSW, K3:8 KEYSW, K3:9 KEYSW, K4:0 KEYSW, K4:1 KEYSW, K4:10 KEYSW, K4:11 KEYSW, K4:13 KEYSW, K4:14 KEYSW, K4:15 KEYSW, K4:16 KEYSW, K4:17 KEYSW, K4:2 KEYSW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

Commit message: added teensy symbol library to replace broken symbol and remapped connections
Parts:
- C1, C2, C_ENC1, C_ENC2, C_REF1, D0:0, D0:1, D0:10, D0:11, D0:12, D0:13, D0:14, D0:15, D0:16, D0:17, D0:2, D0:3, D0:4, D0:5, D0:6, D0:7, D0:8, D0:9, D1:0, D1:1, D1:10, D1:11, D1:12, D1:13, D1:14, D1:15, D1:16, D1:17, D1:2, D1:3, D1:4, D1:5, D1:6, D1:7, D1:8, D1:9, D2:0, D2:1, D2:10, D2:11, D2:12, D2:13, D2:14, D2:15, D2:16, D2:17, D2:2, D2:3, D2:4, D2:5, D2:6, D2:7, D2:8, D2:9, D3:0, D3:1, D3:10, D3:11, D3:12, D3:14, D3:15, D3:16, D3:17, D3:2, D3:3, D3:4, D3:5, D3:6, D3:7, D3:8, D3:9, D4:0, D4:1, D4:10, D4:11, D4:13, D4:14, D4:15, D4:16, D4:17, D4:2, D4:3, D4:4, D4:5, D4:6, D4:7, D4:8, D4:9, D5:0, D5:1, D5:10, D5:12, D5:13, D5:14, D5:15, D5:16, D5:2, D5:5, D5:9, K0:0, K0:1, K0:10, K0:11, K0:12, K0:13, K0:14, K0:15, K0:16, K0:2, K0:3, K0:4, K0:5, K0:6, K0:7, K0:8, K0:9, K1:0, K1:1, K1:10, K1:11, K1:12, K1:13, K1:14, K1:15, K1:16, K1:17, K1:2, K1:3, K1:4, K1:5, K1:6, K1:7, K1:8, K1:9, K2:0, K2:1, K2:10, K2:11, K2:12, K2:13, K2:14, K2:15, K2:16, K2:17, K2:2, K2:3, K2:4, K2:5, K2:6, K2:7, K2:8, K2:9, K3:0, K3:1, K3:10, K3:11, K3:12, K3:14, K3:15, K3:16, K3:17, K3:2, K3:3, K3:4, K3:5, K3:6, K3:7, K3:8, K3:9, K4:0, K4:1, K4:10, K4:11, K4:13, K4:14, K4:15, K4:16, K4:17, K4:2, K4:3, K4:4, K4:5, K4:6, K4:7, K4:8, K4:9, K5:0, K5:1, K5:10, K5:12, K5:13, K5:14, K5:15, K5:16, K5:2, K5:5, K5:9, LED1, LED2, LED3, LED_R1, LED_R2, LED_R3, R1, R2, R_ENC1, R_ENC2, SW1: moved to B.Cu
- U1: value Teensy2.0++ -> Teensy++2.0; moved to B.Cu
- moved U1 539.7 mm to (571.3, 40.6), turned to 270 degrees
- moved D3:10 447.7 mm to (561.9, 367.0)
- moved LED3 446.9 mm to (568.7, 366.6)
- moved D3:8 441.8 mm to (561.9, 363.4)
- moved LED2 439.5 mm to (568.7, 362.0)
- moved D3:1 436.0 mm to (561.9, 359.8)
- moved LED1 432.2 mm to (568.7, 357.5)
- moved D3:0 430.2 mm to (561.9, 356.2)
- moved D2:17 424.5 mm to (561.9, 352.6)
- moved D2:8 418.8 mm to (568.5, 349.0)
- moved D2:6 413.2 mm to (568.5, 345.4)
- moved D2:5 407.6 mm to (568.5, 341.8)
- moved D0:1 402.2 mm to (575.0, 274.0)
- moved D3:15 402.2 mm to (523.0, 274.0)
- moved D2:13 402.2 mm to (554.2, 274.0)
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Connections:
- C_ENC1 pad 2: Net-(C_ENC1-Pad2) -> (no net)
- C_ENC2 pad 1: Net-(C_ENC2-Pad1) -> (no net)
- R_ENC1 pad 1: Net-(R_ENC1-Pad1) -> (no net)
- R_ENC2 pad 1: Net-(R_ENC2-Pad1) -> (no net)
- U1 pad 1: /col7 -> +5V
- U1 pad 10: Net-(U1-Pad10) -> (no net)
- U1 pad 13: Net-(U1-Pad13) -> (no net)
- U1 pad 14: Net-(U1-Pad14) -> (no net)
- U1 pad 15: Net-(U1-Pad15) -> (no net)
- U1 pad 16: Net-(U1-Pad16) -> (no net)
- U1 pad 2: (no net) -> /col7
- U1 pad 20: Net-(U1-Pad20) -> (no net)
- U1 pad 21: /col15 -> VCC
- U1 pad 22: /col14 -> +5V
- U1 pad 23: /col13 -> Net-(R1-Pad2)
- U1 pad 24: /col12 -> /col15
- U1 pad 25: /col11 -> /col14
- U1 pad 26: /col10 -> /col13
- U1 pad 27: /col9 -> /col12
- U1 pad 28: /col8 -> /col11
- U1 pad 29: Net-(C_REF1-Pad2) -> /col10
- U1 pad 30: +5V -> /col9
- U1 pad 31: Net-(U1-Pad31) -> /col8
- U1 pad 32: Net-(U1-Pad32) -> Net-(C_REF1-Pad2)
- U1 pad 33: /col0 -> +5V
- U1 pad 34: /col1 -> (no net)
- U1 pad 35: /col2 -> (no net)
- U1 pad 36: /col3 -> /col0
- U1 pad 37: /col4 -> /col1
- U1 pad 38: /col5 -> /col2
- U1 pad 39: /col6 -> /col3
- U1 pad 40: VCC -> /col4
- U1 pad 41: Net-(U1-Pad41) -> /col5
- U1 pad 42: Net-(U1-Pad42) -> /col6
- U1 pad 43: Net-(U1-Pad43) -> VCC
- U1 pad 44: Net-(U1-Pad44) -> (no net)
- U1 pad 45: Net-(U1-Pad45) -> (no net)
- U1 pad 46: Net-(U1-Pad46) -> (no net)
- U1 pad 47: Net-(U1-Pad47) -> (no net)
- U1 pad 48: Net-(U1-Pad48) -> (no net)
- U1 pad 49: Net-(R2-Pad2) -> (no net)
- U1 pad 50: Net-(U1-Pad50) -> (no net)
- U1 pad 51: Net-(U1-Pad51) -> (no net)
- U1 pad 52: Net-(R1-Pad2) -> Net-(R2-Pad2)
- U1 pad 9: Net-(U1-Pad9) -> (no net)

Commit message: layed out the switch matrix
Parts:
- moved K1:2 426.8 mm to (59.7, 40.7)
- moved K2:0 409.8 mm to (21.7, 60.3)
- moved ENC1 382.7 mm to (339.6, 18.9)
- moved K1:3 382.2 mm to (78.8, 40.6)
- moved K5:16 380.3 mm to (326.6, 116.7)
- moved K4:17 367.1 mm to (345.8, 97.4)
- moved K2:1 364.2 mm to (40.8, 60.3)
- moved K1:10 358.6 mm to (212.0, 40.6)
- moved K4:16 356.3 mm to (326.5, 97.6)
- moved K0:12 352.9 mm to (250.0, 21.6)
- moved K2:17 350.0 mm to (345.4, 59.5)
- moved K5:15 349.6 mm to (307.8, 117.1)
- moved K3:17 349.5 mm to (345.8, 78.6)
- moved K2:16 349.0 mm to (326.2, 59.2)
- moved K1:4 346.3 mm to (97.8, 40.6)
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
Commit message: finished layout. still needs adjustments to schematics to reflect layout
Parts:
- removed K3:17, K5:2: KEYSW, keebs:Mx_Alps_100
- K1:13, K2:17, K4:0, K4:11, K4:17: footprint keebs:Mx_Alps_100 -> keebs:Mx_Alps_200
- K2:0, K2:13, K5:0, K5:1, K5:10, K5:9: footprint keebs:Mx_Alps_100 -> keebs:Mx_Alps_150
- K3:0: footprint keebs:Mx_Alps_100 -> keebs:Mx_Alps_175
- K3:12: footprint keebs:Mx_Alps_100 -> keebs:Mx_Alps_225
- K5:5: footprint keebs:Mx_Alps_100 -> keebs:Mx_Alps_625
- moved C2 301.6 mm to (344.3, -25.1)
- moved D0:14 301.6 mm to (474.4, 13.5)
- moved D0:9 301.6 mm to (457.5, 42.4)
- moved D2:17 301.6 mm to (480.9, 62.1)
- moved D3:2 301.6 mm to (452.4, -23.7)
- moved D3:7 301.6 mm to (442.0, -23.7)
- moved D3:8 301.6 mm to (480.9, 72.9)
- moved D4:10 301.6 mm to (400.4, -23.7)
- moved D5:1 301.6 mm to (379.6, -23.7)
- moved LED2 301.6 mm to (487.8, 71.5)
- moved LED3 301.6 mm to (487.8, 76.1)
- moved C1 301.6 mm to (344.3, -20.9)
- moved C_ENC1 301.6 mm to (344.3, -16.8)
- moved D0:0 301.6 mm to (458.4, 38.8)
- moved D0:1 301.6 mm to (494.0, -16.5)
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
Commit message: switched to keeb.io library and placed diodes
Parts:
- removed D3:17, D5:2: D, keyboard_parts:D_SOD123_axial
- D0:0, D0:1, D0:10, D0:11, D0:12, D0:13, D0:14, D0:15, D0:16, D0:17, D0:2, D0:3, D0:4, D0:5, D0:6, D0:7, D0:8, D0:9, D1:0, D1:1, D1:10, D1:11, D1:12, D1:13, D1:14, D1:15, D1:16, D1:17, D1:2, D1:3, D1:4, D1:5, D1:6, D1:7, D1:8, D1:9, D2:0, D2:1, D2:10, D2:11, D2:12, D2:13, D2:14, D2:15, D2:16, D2:17, D2:2, D2:3, D2:4, D2:5, D2:6, D2:7, D2:8, D2:9, D3:0, D3:1, D3:10, D3:11, D3:12, D3:14, D3:15, D3:16, D3:2, D3:3, D3:4, D3:5, D3:6, D3:7, D3:8, D3:9, D4:0, D4:1, D4:10, D4:11, D4:13, D4:14, D4:15, D4:16, D4:17, D4:2, D4:3, D4:4, D4:5, D4:6, D4:7, D4:8, D4:9, D5:0, D5:1, D5:10, D5:12, D5:13, D5:14, D5:15, D5:16, D5:5, D5:9: footprint keyboard_parts:D_SOD123_axial -> Keebio-Parts:Diode-dual
- K0:0, K0:1, K0:10, K0:11, K0:12, K0:13, K0:14, K0:15, K0:16, K0:2, K0:3, K0:4, K0:5, K0:6, K0:7, K0:8, K0:9, K1:0, K1:1, K1:10, K1:11, K1:12, K1:14, K1:15, K1:16, K1:17, K1:2, K1:3, K1:4, K1:5, K1:6, K1:7, K1:8, K1:9, K2:1, K2:10, K2:11, K2:12, K2:14, K2:15, K2:16, K2:2, K2:3, K2:4, K2:5, K2:6, K2:7, K2:8, K2:9, K3:1, K3:10, K3:11, K3:14, K3:15, K3:16, K3:2, K3:3, K3:4, K3:5, K3:6, K3:7, K3:8, K3:9, K4:1, K4:10, K4:13, K4:14, K4:15, K4:16, K4:2, K4:3, K4:4, K4:5, K4:6, K4:7, K4:8, K4:9, K5:12, K5:13, K5:14, K5:15, K5:16: footprint keebs:Mx_Alps_100 -> Keebio-Parts:Hybrid_PCB_100H_Dual_hole-LED
- K1:13, K2:17, K4:0, K4:11, K4:17: footprint keebs:Mx_Alps_200 -> Keebio-Parts:Hybrid_PCB_200H-dual-LED
- K2:0, K2:13, K5:0, K5:1, K5:10, K5:9: footprint keebs:Mx_Alps_150 -> Keebio-Parts:Hybrid_PCB_100H_Dual_hole-LED
- K3:0: footprint keebs:Mx_Alps_175 -> Keebio-Parts:Hybrid_PCB_100H_Dual_hole-LED
- K3:12: footprint keebs:Mx_Alps_225 -> Keebio-Parts:Hybrid_PCB_200H-dual-LED
- K5:5: footprint keebs:Mx_Alps_625 -> Keebio-Parts:Hybrid_PCB_625H
- SW1: footprint Button_Switch_THT:Push_E-Switch_KS01Q01 -> Keebio-Parts:SW_Tactile_SPST_Angled_MJTP1117
- moved D1:0 484.8 mm to (0.00, 33.3), turned to 270 degrees
- moved D3:0 473.8 mm to (7.14, 71.4), turned to 270 degrees
- moved D0:1 470.9 mm to (23.8, 9.53), turned to 270 degrees
- moved D0:0 459.3 mm to (0.00, 9.53), turned to 270 degrees
- moved D1:2 449.2 mm to (38.1, 33.3), turned to 270 degrees
- moved D3:1 447.6 mm to (33.3, 71.4), turned to 270 degrees
- moved D0:2 445.7 mm to (42.9, 9.53), turned to 270 degrees
- moved D2:0 443.5 mm to (4.76, 52.4), turned to 270 degrees
- moved D4:0 435.4 mm to (9.53, 90.5), turned to 270 degrees
- moved D1:1 432.8 mm to (19.1, 33.3), turned to 270 degrees
- moved D2:1 429.0 mm to (28.6, 52.4), turned to 270 degrees
- moved D0:3 427.0 mm to (61.9, 9.53), turned to 270 degrees
- moved D2:3 420.8 mm to (66.7, 52.4), turned to 270 degrees
- moved D3:2 411.2 mm to (52.4, 71.4), turned to 270 degrees
- moved D1:4 410.9 mm to (76.2, 33.3), turned to 270 degrees
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Connections:
- C_ENC1 pad 2: (no net) -> Net-(C_ENC1-Pad2)
- C_ENC2 pad 1: (no net) -> Net-(C_ENC2-Pad1)
- R_ENC1 pad 1: (no net) -> Net-(C_ENC1-Pad2)
- R_ENC2 pad 1: (no net) -> Net-(C_ENC2-Pad1)
- U1 pad 10: (no net) -> Net-(U1-Pad10)
- U1 pad 13: (no net) -> Net-(U1-Pad13)
- U1 pad 14: (no net) -> Net-(U1-Pad14)
- U1 pad 15: (no net) -> Net-(U1-Pad15)
- U1 pad 16: (no net) -> Net-(U1-Pad16)
- U1 pad 20: (no net) -> Net-(U1-Pad20)
- U1 pad 34: (no net) -> Net-(U1-Pad34)
- U1 pad 35: (no net) -> Net-(U1-Pad35)
- U1 pad 44: (no net) -> Net-(U1-Pad44)
- U1 pad 45: (no net) -> Net-(U1-Pad45)
- U1 pad 46: (no net) -> Net-(U1-Pad46)
- U1 pad 47: (no net) -> Net-(U1-Pad47)
- U1 pad 48: (no net) -> Net-(U1-Pad48)
- U1 pad 49: (no net) -> Net-(U1-Pad49)
- U1 pad 50: (no net) -> Net-(U1-Pad50)
- U1 pad 51: (no net) -> Net-(U1-Pad51)
- U1 pad 9: (no net) -> Net-(U1-Pad9)

Commit message: fixed +5v vs GND discrepency. More routing.
Parts:
- moved U1 287.7 mm to (9.53, 19.1)
- moved R1 219.1 mm to (66.7, 0.00), turned to 180 degrees
- moved C1 214.3 mm to (66.7, -4.76)
- moved C_REF1 211.6 mm to (-2.38, 19.1), turned to 270 degrees
- moved SW1 208.9 mm to (81.0, 0.00)
- moved R2 202.6 mm to (1.50, 55.5), turned to 90 degrees
- moved C2 201.6 mm to (69.1, 0.00)
- moved LED3 86.1 mm to (323.9, -1.99), turned to 90 degrees
- moved LED_R3 81.4 mm to (319.1, -4.76), turned to 270 degrees
- moved LED2 67.5 mm to (309.6, -1.99), turned to 90 degrees
- moved LED_R2 63.5 mm to (304.8, -4.76), turned to 270 degrees
- moved LED_R1 57.2 mm to (290.5, -4.76), turned to 270 degrees
- moved LED1 50.2 mm to (295.3, -1.99), turned to 90 degrees
- moved D1:0 25.6 mm to (23.8, 23.8), turned to 0 degrees
- moved D0:0 21.4 mm to (21.4, 9.53)
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Connections:
- C_ENC1 pad 1: +5V -> GND
- C_ENC2 pad 2: +5V -> GND
- C_REF1 pad 1: +5V -> GND
- ENC1 pad C: +5V -> GND
- U1 pad 1: +5V -> GND
- U1 pad 10: Net-(U1-Pad10) -> (no net)
- U1 pad 13: Net-(U1-Pad13) -> (no net)
- U1 pad 14: Net-(U1-Pad14) -> (no net)
- U1 pad 15: Net-(U1-Pad15) -> (no net)
- U1 pad 16: Net-(U1-Pad16) -> (no net)
- U1 pad 20: Net-(U1-Pad20) -> (no net)
- U1 pad 22: +5V -> GND
- U1 pad 33: +5V -> GND
- U1 pad 34: Net-(U1-Pad34) -> (no net)
- U1 pad 35: Net-(U1-Pad35) -> (no net)
- U1 pad 44: Net-(U1-Pad44) -> (no net)
- U1 pad 45: Net-(U1-Pad45) -> (no net)
- U1 pad 46: Net-(U1-Pad46) -> (no net)
- U1 pad 47: Net-(U1-Pad47) -> (no net)
- U1 pad 48: Net-(U1-Pad48) -> (no net)
- U1 pad 49: Net-(U1-Pad49) -> (no net)
- U1 pad 50: Net-(U1-Pad50) -> (no net)
- U1 pad 51: Net-(U1-Pad51) -> (no net)
- U1 pad 9: Net-(U1-Pad9) -> (no net)
Routing:
- net /col15: track 0.00 -> 489.5 mm, vias 0 -> 1
- net /row4: track 0.00 -> 483.1 mm
- net /col17: track 0.00 -> 449.8 mm, vias 0 -> 3
- net /row5: track 0.00 -> 445.3 mm
- net /col16: track 0.00 -> 425.1 mm, vias 0 -> 3
- net /row3: track 0.00 -> 409.5 mm, vias 0 -> 1
- net /row2: track 0.00 -> 407.9 mm
- net /row1: track 0.00 -> 374.3 mm
- net /row0: track 0.00 -> 347.6 mm
- net /col7: track 0.00 -> 237.2 mm
- net VCC: track 0.00 -> 138.7 mm
- net /col12: track 0.00 -> 123.7 mm
- net /col10: track 0.00 -> 117.1 mm
- net Net-(R1-Pad2): track 0.00 -> 114.0 mm, vias 0 -> 5
- net /col13: track 0.00 -> 112.1 mm
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- added copper zone on B.Cu, net GND
- added copper zone on F.Cu, net GND
Other:
- board outline added: 381 x 133.3 mm
