File: CBC2.kicad_pcb (KiCad board)
At the start: 2 copper layers, 381 x 133.3 mm, 211 parts, among them K0:0 KEYSW, K0:1 KEYSW, K0:10 KEYSW, K0:11 KEYSW, K0:12 KEYSW, K0:13 KEYSW, K0:14 KEYSW, K0:15 KEYSW, K0:16 KEYSW, K0:2 KEYSW, K0:3 KEYSW, K0:4 KEYSW, K0:5 KEYSW, K0:6 KEYSW, K0:7 KEYSW, K0:8 KEYSW, K0:9 KEYSW, K1:0 KEYSW, K1:1 KEYSW, K1:10 KEYSW, K1:11 KEYSW, K1:12 KEYSW, K1:13 KEYSW, K1:14 KEYSW, K1:15 KEYSW, K1:16 KEYSW, K1:17 KEYSW, K1:2 KEYSW, K1:3 KEYSW, K1:4 KEYSW, K1:5 KEYSW, K1:6 KEYSW, K1:7 KEYSW, K1:8 KEYSW, K1:9 KEYSW, K2:0 KEYSW, K2:1 KEYSW, K2:10 KEYSW, K2:11 KEYSW, K2:12 KEYSW, K2:13 KEYSW, K2:14 KEYSW, K2:15 KEYSW, K2:16 KEYSW, K2:17 KEYSW, K2:2 KEYSW, K2:3 KEYSW, K2:4 KEYSW, K2:5 KEYSW, K2:6 KEYSW, K2:7 KEYSW, K2:8 KEYSW, K2:9 KEYSW, K3:0 KEYSW, K3:1 KEYSW, K3:10 KEYSW, K3:11 KEYSW, K3:12 KEYSW, K3:14 KEYSW, K3:15 KEYSW, K3:16 KEYSW, K3:2 KEYSW, K3:3 KEYSW, K3:4 KEYSW, K3:5 KEYSW, K3:6 KEYSW, K3:7 KEYSW, K3:8 KEYSW, K3:9 KEYSW, K4:0 KEYSW, K4:1 KEYSW, K4:10 KEYSW, K4:11 KEYSW, K4:13 KEYSW, K4:14 KEYSW, K4:15 KEYSW, K4:16 KEYSW, K4:17 KEYSW, K4:2 KEYSW, K4:3 KEYSW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

Commit message: final touches
Parts:
- added U4: HOLE, Keebio-Parts:MountingHole, F.Cu at (2.00, 68.0)
- added U4: HOLE, Keebio-Parts:MountingHole, F.Cu at (290.0, 65.0)
- added U4: HOLE, Keebio-Parts:MountingHole, F.Cu at (162.5, -5.00)
- added U4: HOLE, Keebio-Parts:MountingHole, F.Cu at (347.5, -5.00)
- added U4: HOLE, Keebio-Parts:MountingHole, F.Cu at (365.0, 117.5)
- added U4: HOLE, Keebio-Parts:MountingHole, F.Cu at (245.0, 117.5)
- added U4: HOLE, Keebio-Parts:MountingHole, F.Cu at (115.0, 117.5)
- added U4: HOLE, Keebio-Parts:MountingHole, F.Cu at (2.50, 117.5)
- moved C_ENC2 7.14 mm to (361.9, 0.00), turned to 180 degrees
Routing:
- net /led3: track 0.00 -> 373.5 mm, vias 0 -> 1
- net /led2: track 0.00 -> 325.8 mm, vias 0 -> 1
- net /led1: track 0.00 -> 310.8 mm, vias 0 -> 3
- net Net-(ENC1-PadB): track 0.00 -> 7.05 mm
- net Net-(ENC1-PadA): track 0.00 -> 7.03 mm
- net Net-(D3:3-Pad2): track 0.00 -> 5.73 mm
- net Net-(LED3-Pad1): track 0.00 -> 5.72 mm
- net Net-(LED2-Pad1): track 0.00 -> 5.72 mm
- net Net-(LED1-Pad1): track 0.00 -> 5.72 mm
- net Net-(C_ENC2-Pad1): track 0.00 -> 2.38 mm
- net Net-(C_ENC1-Pad2): track 0.00 -> 2.03 mm
- net /row1: track 374.3 -> 375.7 mm
- net Net-(R1-Pad2): track 117.8 -> 119.1 mm
- net /col13: track 386.9 -> 387.9 mm
- net /col2: track 150.3 -> 151.2 mm
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Other:
- board text added: "Tim Bretz"

Commit message: i lied. started the pcb from scratch after modifying schematic and layout plans
Parts:
- removed D0:16, D4:1, D4:13, D5:1, D5:10, D5:5, D5:9: D, Keebio-Parts:Diode-dual
- removed K0:16, K4:1, K4:13, K5:1, K5:10, K5:9: KEYSW, Keebio-Parts:Hybrid_PCB_100H_Dual_hole-LED
- removed K5:5: KEYSW, Keebio-Parts:Hybrid_PCB_625H
- removed LED1, LED2, LED3: LED, LED_THT:LED_D2.0mm_W4.0mm_H2.8mm_FlatTop
- removed LED_R1, LED_R2, LED_R3: 1k, Resistor_THT:R_Axial_DIN0204_L3.6mm_D1.6mm_P5.08mm_Horizontal
- removed U4 (x8): HOLE, Keebio-Parts:MountingHole
- added D1:18: D, Keebio-Parts:Diode-dual, F.Cu at (303.1, 183.4)
- added D2:18: D, Keebio-Parts:Diode-dual, F.Cu at (323.3, 155.2)
- added D3:17: D, Keebio-Parts:Diode-dual, F.Cu at (447.5, 161.5)
- added D4:12: D, Keebio-Parts:Diode-dual, F.Cu at (447.5, 164.2)
- added D4:18: D, Keebio-Parts:Diode-dual, F.Cu at (447.5, 166.9)
- added D5:11: D, Keebio-Parts:Diode-dual, F.Cu at (288.0, 173.8)
- added D5:17: D, Keebio-Parts:Diode-dual, F.Cu at (447.5, 169.5)
- added D5:2: D, Keebio-Parts:Diode-dual, F.Cu at (62.2, -19.1)
- added D5:7: D, Keebio-Parts:Diode-dual, F.Cu at (162.6, -19.1)
- added K1:18: KEYSW, MX_Alps_Hybrid:MX-1U, F.Cu at (376.2, 33.3)
- added K2:18: KEYSW, MX_Alps_Hybrid:MX-2U, F.Cu at (376.2, 61.9)
- added K3:17: KEYSW, MX_Alps_Hybrid:MX-1U, F.Cu at (357.2, 71.4)
- added K4:12: KEYSW, MX_Alps_Hybrid:MX-2.5U, F.Cu at (257.2, 90.5)
- added K4:18: KEYSW, MX_Alps_Hybrid:MX-2U, F.Cu at (376.2, 100.0)
- added K5:11: KEYSW, MX_Alps_Hybrid:MX-1.5U, F.Cu at (219.1, 109.5)
- added K5:17: KEYSW, MX_Alps_Hybrid:MX-1U, F.Cu at (357.2, 109.5)
- added K5:2: KEYSW, MX_Alps_Hybrid:MX-1.5U, F.Cu at (57.1, 109.5)
- added K5:7: KEYSW, MX_Alps_Hybrid:MX-7U, F.Cu at (138.1, 109.5)
- C1, C2, C_ENC1, C_ENC2, C_REF1, D0:0, D0:1, D0:10, D0:11, D0:12, D0:13, D0:14, D0:15, D0:17, D0:2, D0:3, D0:4, D0:5, D0:6, D0:7, D0:8, D0:9, D1:0, D1:1, D1:10, D1:11, D1:12, D1:13, D1:14, D1:15, D1:16, D1:17, D1:2, D1:3, D1:4, D1:5, D1:6, D1:7, D1:8, D1:9, D2:0, D2:1, D2:10, D2:11, D2:12, D2:13, D2:14, D2:15, D2:16, D2:17, D2:2, D2:3, D2:4, D2:5, D2:6, D2:7, D2:8, D2:9, D3:0, D3:1, D3:10, D3:11, D3:12, D3:14, D3:15, D3:16, D3:2, D3:3, D3:4, D3:5, D3:6, D3:7, D3:8, D3:9, D4:0, D4:10, D4:11, D4:14, D4:15, D4:16, D4:17, D4:2, D4:3, D4:4, D4:5, D4:6, D4:7, D4:8, D4:9, D5:0, D5:12, D5:13, D5:14, D5:15, D5:16, R1, R2, R_ENC1, R_ENC2, SW1, U1: moved to F.Cu
- K0:0, K0:1, K0:10, K0:11, K0:12, K0:13, K0:14, K0:15, K0:2, K0:3, K0:4, K0:5, K0:6, K0:7, K0:8, K0:9, K1:0, K1:1, K1:10, K1:11, K1:12, K1:14, K1:15, K1:16, K1:17, K1:2, K1:3, K1:4, K1:5, K1:6, K1:7, K1:8, K1:9, K2:1, K2:10, K2:11, K2:12, K2:14, K2:15, K2:16, K2:2, K2:3, K2:4, K2:5, K2:6, K2:7, K2:8, K2:9, K3:1, K3:10, K3:11, K3:14, K3:15, K3:16, K3:2, K3:3, K3:4, K3:5, K3:6, K3:7, K3:8, K3:9, K4:10, K4:14, K4:15, K4:16, K4:2, K4:3, K4:4, K4:5, K4:6, K4:7, K4:8, K4:9, K5:13, K5:14, K5:15, K5:16: footprint Keebio-Parts:Hybrid_PCB_100H_Dual_hole-LED -> MX_Alps_Hybrid:MX-1U; moved to F.Cu
- K1:13: footprint Keebio-Parts:Hybrid_PCB_200H-dual-LED -> MX_Alps_Hybrid:MX-1.75U; moved to F.Cu
- K2:0, K5:0, K5:12: footprint Keebio-Parts:Hybrid_PCB_100H_Dual_hole-LED -> MX_Alps_Hybrid:MX-1.5U; moved to F.Cu
- K2:13: footprint Keebio-Parts:Hybrid_PCB_100H_Dual_hole-LED -> MX_Alps_Hybrid:MX-1.25U; moved to F.Cu
- K2:17, K4:11, K4:17: footprint Keebio-Parts:Hybrid_PCB_200H-dual-LED -> MX_Alps_Hybrid:MX-1U; moved to F.Cu
- K3:0: footprint Keebio-Parts:Hybrid_PCB_100H_Dual_hole-LED -> MX_Alps_Hybrid:MX-1.75U; moved to F.Cu
- K3:12: footprint Keebio-Parts:Hybrid_PCB_200H-dual-LED -> MX_Alps_Hybrid:MX-2U; moved to F.Cu
- K4:0: footprint Keebio-Parts:Hybrid_PCB_200H-dual-LED -> MX_Alps_Hybrid:MX-2.25U; moved to F.Cu
- moved U1 367.3 mm to (376.2, -2.38)
- moved R2 361.2 mm to (352.6, 140.6), turned to 0 degrees
- moved C_ENC2 333.6 mm to (93.9, 198.5), turned to 0 degrees
- moved C_ENC1 319.1 mm to (93.9, 202.7)
- moved D4:15 311.5 mm to (59.1, 269.0), turned to 0 degrees
- moved R1 304.4 mm to (307.0, 186.8), turned to 0 degrees
- moved D4:17 303.8 mm to (72.5, 184.5), turned to 0 degrees
- moved D4:16 277.9 mm to (121.5, 270.3), turned to 0 degrees
- moved C2 272.0 mm to (34.4, 269.8)
- moved D1:17 244.8 mm to (240.0, 250.8), turned to 0 degrees
- moved D3:16 244.4 mm to (190.4, 269.6), turned to 0 degrees
- moved D4:14 236.1 mm to (142.3, 270.3), turned to 0 degrees
- moved D0:12 224.1 mm to (260.2, 233.3), turned to 0 degrees
- moved SW1 221.4 mm to (190.1, 192.6)
- moved D0:11 218.2 mm to (269.8, 223.8), turned to 0 degrees
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Connections:
- K1:16 pad 1: /col16 -> Net-(K1:16-Pad1)
- K2:16 pad 1: /col16 -> Net-(K1:16-Pad1)
- K3:16 pad 1: /col16 -> Net-(K1:16-Pad1)
- K4:16 pad 1: /col16 -> Net-(K1:16-Pad1)
- K5:16 pad 1: /col16 -> Net-(K1:16-Pad1)
- U1 pad 11: /col16 -> (no net)
- U1 pad 13: (no net) -> /col18
- U1 pad 17: /led1 -> (no net)
- U1 pad 18: /led2 -> (no net)
- U1 pad 19: /led3 -> (no net)
Routing:
- net /col15: track 471.3 -> 0.00 mm, vias 1 -> 0
- net /row4: track 459.5 -> 0.00 mm, vias 1 -> 0
- net /col14: track 458.2 -> 0.00 mm, vias 1 -> 0
- net /row5: track 453.3 -> 0.00 mm
- net /col17: track 450.4 -> 0.00 mm, vias 3 -> 0
- net /col16: track 425.1 -> 0.00 mm, vias 3 -> 0
- net /row2: track 409.8 -> 0.00 mm
- net /row3: track 409.5 -> 0.00 mm, vias 1 -> 0
- net /col13: track 387.9 -> 0.00 mm, vias 1 -> 0
- net /col12: track 386.0 -> 0.00 mm, vias 1 -> 0
- net /row1: track 375.7 -> 0.00 mm
- net /led3: track 373.5 -> 0.00 mm, vias 1 -> 0
- net /col10: track 366.6 -> 0.00 mm, vias 1 -> 0
- net /col11: track 363.6 -> 0.00 mm, vias 1 -> 0
- net /col9: track 355.8 -> 0.00 mm, vias 1 -> 0
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- removed copper zone on B.Cu, net GND
- removed copper zone on F.Cu, net GND
Other:
- board outline removed
- board text removed: "Tim Bretz"

Commit message: updated footprints for layout adjustment. placed diodes, still on the fence about the microcontroller placement
Parts:
- C1, C2, C_ENC1, C_ENC2, C_REF1, D0:0, D0:1, D0:10, D0:11, D0:12, D0:13, D0:14, D0:15, D0:17, D0:2, D0:3, D0:4, D0:5, D0:6, D0:7, D0:8, D0:9, D1:0, D1:1, D1:10, D1:11, D1:12, D1:13, D1:14, D1:15, D1:16, D1:17, D1:18, D1:2, D1:3, D1:4, D1:5, D1:6, D1:7, D1:8, D1:9, D2:0, D2:1, D2:10, D2:11, D2:12, D2:13, D2:14, D2:15, D2:16, D2:17, D2:18, D2:2, D2:3, D2:4, D2:5, D2:6, D2:7, D2:8, D2:9, D3:0, D3:1, D3:10, D3:11, D3:12, D3:14, D3:15, D3:16, D3:17, D3:2, D3:3, D3:4, D3:5, D3:6, D3:7, D3:8, D3:9, D4:0, D4:10, D4:11, D4:12, D4:14, D4:15, D4:16, D4:17, D4:18, D4:2, D4:3, D4:4, D4:5, D4:6, D4:7, D4:8, D4:9, D5:0, D5:11, D5:12, D5:13, D5:14, D5:15, D5:16, D5:17, D5:2, D5:7, R1, R2, R_ENC1, R_ENC2, SW1, U1: moved to B.Cu
- K1:13: footprint MX_Alps_Hybrid:MX-1.75U -> MX_Alps_Hybrid:MX-2U
- K2:13: footprint MX_Alps_Hybrid:MX-1.25U -> MX_Alps_Hybrid:MX-1.5U
- K3:12: footprint MX_Alps_Hybrid:MX-2U -> MX_Alps_Hybrid:MX-2.25U
- K4:12: footprint MX_Alps_Hybrid:MX-2.5U -> MX_Alps_Hybrid:MX-2.75U
- moved U1 352.5 mm to (23.8, -9.53), turned to 0 degrees
- moved D4:15 327.3 mm to (333.4, 90.5), turned to 270 degrees
- moved C_ENC1 326.7 mm to (350.0, 0.00), turned to 180 degrees
- moved R2 318.0 mm to (76.2, -16.7), turned to 180 degrees
- moved D4:17 313.4 mm to (371.5, 90.5), turned to 270 degrees
- moved C_ENC2 305.6 mm to (342.9, 21.4)
- moved R1 299.0 mm to (85.7, -14.3)
- moved D4:16 292.7 mm to (352.4, 90.5), turned to 270 degrees
- moved C2 287.3 mm to (57.1, -16.7)
- moved D3:16 256.0 mm to (352.4, 71.4), turned to 270 degrees
- moved D1:17 254.1 mm to (371.5, 33.3), turned to 270 degrees
- moved D4:14 242.1 mm to (309.6, 95.2), turned to 270 degrees
- moved SW1 233.9 mm to (90.5, -19.1), turned to 180 degrees
- moved D0:12 223.9 mm to (266.7, 9.53), turned to 270 degrees
- moved D5:13 219.2 mm to (290.5, 114.3), turned to 270 degrees
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Connections:
- D5:7 pad 2: /col6 -> Net-(D5:7-Pad2)
- K5:7 pad 2: Net-(K5:7-Pad2) -> Net-(D5:7-Pad2)
- U1 pad 10: (no net) -> Net-(U1-Pad10)
- U1 pad 11: (no net) -> /col16
- U1 pad 14: (no net) -> Net-(U1-Pad14)
- U1 pad 15: (no net) -> Net-(U1-Pad15)
- U1 pad 16: (no net) -> Net-(U1-Pad16)
- U1 pad 17: (no net) -> Net-(U1-Pad17)
- U1 pad 18: (no net) -> Net-(U1-Pad18)
- U1 pad 19: (no net) -> Net-(U1-Pad19)
- U1 pad 20: (no net) -> Net-(U1-Pad20)
- U1 pad 34: (no net) -> Net-(U1-Pad34)
- U1 pad 35: (no net) -> Net-(U1-Pad35)
- U1 pad 44: (no net) -> Net-(U1-Pad44)
- U1 pad 45: (no net) -> Net-(U1-Pad45)
- U1 pad 46: (no net) -> Net-(U1-Pad46)
- U1 pad 47: (no net) -> Net-(U1-Pad47)
- U1 pad 48: (no net) -> Net-(U1-Pad48)
- U1 pad 49: (no net) -> Net-(U1-Pad49)
- U1 pad 50: (no net) -> Net-(U1-Pad50)
- U1 pad 51: (no net) -> Net-(U1-Pad51)
- U1 pad 9: (no net) -> Net-(U1-Pad9)
