File: _autosave-CBC2.kicad_pcb (KiCad board)
At the start: 2 copper layers, 381 x 133.3 mm, 211 parts, among them K0:0 KEYSW, K0:1 KEYSW, K0:10 KEYSW, K0:11 KEYSW, K0:12 KEYSW, K0:13 KEYSW, K0:14 KEYSW, K0:15 KEYSW, K0:16 KEYSW, K0:2 KEYSW, K0:3 KEYSW, K0:4 KEYSW, K0:5 KEYSW, K0:6 KEYSW, K0:7 KEYSW, K0:8 KEYSW, K0:9 KEYSW, K1:0 KEYSW, K1:1 KEYSW, K1:10 KEYSW, K1:11 KEYSW, K1:12 KEYSW, K1:13 KEYSW, K1:14 KEYSW, K1:15 KEYSW, K1:16 KEYSW, K1:17 KEYSW, K1:2 KEYSW, K1:3 KEYSW, K1:4 KEYSW, K1:5 KEYSW, K1:6 KEYSW, K1:7 KEYSW, K1:8 KEYSW, K1:9 KEYSW, K2:0 KEYSW, K2:1 KEYSW, K2:10 KEYSW, K2:11 KEYSW, K2:12 KEYSW, K2:13 KEYSW, K2:14 KEYSW, K2:15 KEYSW, K2:16 KEYSW, K2:17 KEYSW, K2:2 KEYSW, K2:3 KEYSW, K2:4 KEYSW, K2:5 KEYSW, K2:6 KEYSW, K2:7 KEYSW, K2:8 KEYSW, K2:9 KEYSW, K3:0 KEYSW, K3:1 KEYSW, K3:10 KEYSW, K3:11 KEYSW, K3:12 KEYSW, K3:14 KEYSW, K3:15 KEYSW, K3:16 KEYSW, K3:2 KEYSW, K3:3 KEYSW, K3:4 KEYSW, K3:5 KEYSW, K3:6 KEYSW, K3:7 KEYSW, K3:8 KEYSW, K3:9 KEYSW, K4:0 KEYSW, K4:1 KEYSW, K4:10 KEYSW, K4:11 KEYSW, K4:13 KEYSW, K4:14 KEYSW, K4:15 KEYSW, K4:16 KEYSW, K4:17 KEYSW, K4:2 KEYSW, K4:3 KEYSW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

Commit message: almost done routing. still needs DRC
Parts:
- moved C_ENC2 7.44 mm to (362.2, 0.00), turned to 180 degrees
Routing:
- net /led3: track 0.00 -> 350.4 mm, vias 0 -> 1
- net /led2: track 0.00 -> 325.8 mm, vias 0 -> 1
- net /led1: track 0.00 -> 313.7 mm, vias 0 -> 3
- net Net-(ENC1-PadB): track 0.00 -> 7.05 mm
- net Net-(ENC1-PadA): track 0.00 -> 7.03 mm
- net Net-(C_ENC1-Pad2): track 0.00 -> 2.03 mm
- net /row1: track 374.3 -> 375.5 mm
- net /col13: track 386.9 -> 387.9 mm
- net Net-(R1-Pad2): track 117.8 -> 118.8 mm
- net /col2: track 150.3 -> 151.2 mm
